File: GateDrive.sch (KiCad schematic (older format))
At the start: 34 parts, among them U2 TLP152, U3 TLP152, U4 TLP152, U5 TLP152, U6 TLP152, U7 TLP152, U8 TLP152

Commit message: テストポイント追加，シルク調整，固定穴マスク追加
Parts:
- added TP10, TP11, TP12, TP6, TP7, TP8, TP9: TestPoint, TestPoint:TestPoint_Pad_D1.0mm, symbol Connector:TestPoint
Connections:
- net SIG_BR: now also TP8.1
- net SIG_UN: now also TP7.1
- net SIG_UP: now also TP6.1
- net SIG_VN: now also TP10.1
- net SIG_VP: now also TP9.1
- net SIG_WN: now also TP12.1
- net SIG_WP: now also TP11.1
Changed lines of the file:
@@
 	1600 3950 1350 3950
 Wire Wire Line
-	1150 1950 1000 1950
-Wire Wire Line
-	1150 3950 1000 3950
+	1150 1950 1100 1950
+Wire Wire Line
+	1150 3950 1100 3950
 $Comp
 L tlp152:TLP152 U5
@@
 	5100 3950 4850 3950
 Wire Wire Line
-	4650 1950 4500 1950
-Wire Wire Line
-	4650 3950 4500 3950
+	4650 1950 4600 1950
+Wire Wire Line
+	4650 3950 4600 3950
 $Comp
 L tlp152:TLP152 U7
@@
 	8600 3950 8350 3950
 Wire Wire Line
-	8150 1950 8000 1950
-Wire Wire Line
-	8150 3950 8000 3950
+	8150 1950 8100 1950
+Wire Wire Line
+	8150 3950 8100 3950
 Text HLabel 3000 4550 2    50   UnSpc ~ 0
 SOURCE_UN
@@
 	1600 5950 1350 5950
 Wire Wire Line
-	1150 5950 1000 5950
+	1150 5950 1100 5950
 Text HLabel 3000 6550 2    50   UnSpc ~ 0
 SOURCE_BR
@@
 	1    0    0    -1
 $EndComp
+$Comp
+L Connector:TestPoint TP6
+U 1 1 5EC5B30A
+P 1100 1850
+F 0 "TP6" H 850 2000 50  0000 L CNN
+F 1 "TestPoint" H 700 1900 50  0000 L CNN
+F 2 "TestPoint:TestPoint_Pad_D1.0mm" H 1300 1850 50  0001 C CNN
+F 3 "~" H 1300 1850 50  0001 C CNN
+	1    1100 1850
+	1    0    0    -1
+$EndComp
+Wire Wire Line
+	1100 1850 1100 1950
+Connection ~ 1100 1950
+Wire Wire Line
+	1100 1950 1000 1950
+$Comp
+L Connector:TestPoint TP7
+U 1 1 5EC5FE11
+P 1100 3850
+F 0 "TP7" H 850 4000 50  0000 L CNN
+F 1 "TestPoint" H 700 3900 50  0000 L CNN
+F 2 "TestPoint:TestPoint_Pad_D1.0mm" H 1300 3850 50  0001 C CNN
+F 3 "~" H 1300 3850 50  0001 C CNN
+	1    1100 3850
+	1    0    0    -1
+$EndComp
+Wire Wire Line
+	1100 3850 1100 3950
+Connection ~ 1100 3950
+Wire Wire Line
+	1100 3950 1000 3950
+$Comp
+L Connector:TestPoint TP8
+U 1 1 5EC68358
+P 1100 5850
+F 0 "TP8" H 850 6000 50  0000 L CNN
+F 1 "TestPoint" H 700 5900 50  0000 L CNN
+F 2 "TestPoint:TestPoint_Pad_D1.0mm" H 1300 5850 50  0001 C CNN
+F 3 "~" H 1300 5850 50  0001 C CNN
+	1    1100 5850
+	1    0    0    -1
+$EndComp
+Wire Wire Line
+	1100 5850 1100 5950
+Connection ~ 1100 5950
+Wire Wire Line
+	1100 5950 1000 5950
+$Comp
+L Connector:TestPoint TP9
+U 1 1 5EC6EDBA
+P 4600 1850
+F 0 "TP9" H 4350 2000 50  0000 L CNN
+F 1 "TestPoint" H 4200 1900 50  0000 L CNN
+F 2 "TestPoint:TestPoint_Pad_D1.0mm" H 4800 1850 50  0001 C CNN
+F 3 "~" H 4800 1850 50  0001 C CNN
+	1    4600 1850
+	1    0    0    -1
+$EndComp
+Wire Wire Line
+	4600 1850 4600 1950
+Connection ~ 4600 1950
+Wire Wire Line
+	4600 1950 4500 1950
+$Comp
+L Connector:TestPoint TP10
+U 1 1 5EC75D3A
+P 4600 3850
+F 0 "TP10" H 4350 4000 50  0000 L CNN
+F 1 "TestPoint" H 4200 3900 50  0000 L CNN
+F 2 "TestPoint:TestPoint_Pad_D1.0mm" H 4800 3850 50  0001 C CNN
+F 3 "~" H 4800 3850 50  0001 C CNN
+	1    4600 3850
+	1    0    0    -1
+$EndComp
+Wire Wire Line
+	4600 3850 4600 3950
+Connection ~ 4600 3950
+Wire Wire Line
+	4600 3950 4500 3950
+$Comp
+L Connector:TestPoint TP11
+U 1 1 5EC7CDA9
+P 8100 1850
+F 0 "TP11" H 7850 2000 50  0000 L CNN
+F 1 "TestPoint" H 7700 1900 50  0000 L CNN
+F 2 "TestPoint:TestPoint_Pad_D1.0mm" H 8300 1850 50  0001 C CNN
+F 3 "~" H 8300 1850 50  0001 C CNN
+	1    8100 1850
+	1    0    0    -1
+$EndComp
+Wire Wire Line
+	8100 1850 8100 1950
+Connection ~ 8100 1950
+Wire Wire Line
+	8100 1950 8000 1950
+$Comp
+L Connector:TestPoint TP12
+U 1 1 5EC8412B
+P 8100 3850
+F 0 "TP12" H 7850 4000 50  0000 L CNN
+F 1 "TestPoint" H 7700 3900 50  0000 L CNN
+F 2 "TestPoint:TestPoint_Pad_D1.0mm" H 8300 3850 50  0001 C CNN
+F 3 "~" H 8300 3850 50  0001 C CNN
+	1    8100 3850
+	1    0    0    -1
+$EndComp
+Wire Wire Line
+	8100 3850 8100 3950
+Connection ~ 8100 3950
+Wire Wire Line
+	8100 3950 8000 3950
 $EndSCHEMATC
